File: Project/PCB/smartEggTimer/smartEggTimer.kicad_sch (KiCad schematic)
At the start: 65 parts, among them J1 Conn_01x05_Pin, J2 Conn_01x03_Pin, J3 Conn_01x03_Pin, J4 Conn_01x06_Pin, J5 Conn_01x02_Socket, J6 Conn_01x02_Socket, J7 Conn_01x03_Pin, J8 Conn_01x03_Pin, Q2 STP60NF06L, SW1 SW_Push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

Commit message: finish PCB routing Further changes: - Change schematic symbol of MOSFET s.t. pin assignment is correct - Add STEP file for DFPlayer Mini - Save edited footprints to custom-parts project library - Set "exclude from BOM" attribute for components which will be soldered manually
Parts:
- H1, H2: footprint MountingHole:MountingHole_4.3mm_M4 -> custom-parts:MountingHole_4.3mm_M4_Without-Screws
- H3, H8: footprint MountingHole:MountingHole_4.3mm_M4_DIN965 -> custom-parts:MountingHole_4.3mm_M4_Without-Screws
- J1, J2, J3, J4, J5, J6, J7, J8, OLED-15W-C1, SW1, SW3, SW4: now left out of the parts list
- Q1: renamed from Q2; now left out of the parts list
- SW2: footprint Rotary_Encoder:RotaryEncoder_Alps_EC12E_Vertical_H20mm -> custom-parts:RotaryEncoder_Alps_EC12E_Vertical_H20mm_Mounting-Holes-GND
- SW5: footprint Button_Switch_THT:SW_PUSH_6mm_H13mm -> custom-parts:SW_PUSH_6mm_H13mm_No-Pad_Top-Right; now left out of the parts list
- SW6: footprint Button_Switch_THT:SW_PUSH_6mm_H13mm -> custom-parts:SW_PUSH_6mm_H13mm_No-Pad_Top-Left; now left out of the parts list
- SW7: footprint Button_Switch_THT:SW_Slide_SPDT_Angled_CK_OS102011MA1Q -> custom-parts:SW_Slide_SPDT_Angled_CK_OS102011MA1Q_Protruding; now left out of the parts list
- renumbered U3 to U2
Connections:
- net SPK+: now also J5.2 (Pin_2); no longer J5.1 (Pin_1)
- net SPK-: now also J5.1 (Pin_1); no longer J5.2 (Pin_2)
- net DFPlayer-Minus: now reaches DFPlayerMini1.10 (GND), DFPlayerMini1.7 (GND), Q1.2 (D)
Changed lines of the file:
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@@
 	)
 	(label "SPK+"
-		(at 346.71 85.09 180)
+		(at 346.71 87.63 180)
 		(fields_autoplaced yes)
 		(effects
@@
 	)
 	(label "SPK-"
-		(at 346.71 87.63 180)
+		(at 346.71 85.09 180)
 		(fields_autoplaced yes)
 		(effects
@@
 		)
 	)
+	(label "DFPlayer-Minus"
+		(at 53.34 193.04 0)
+		(fields_autoplaced yes)
+		(effects
+			(font
+				(size 1.27 1.27)
+			)
+			(justify left bottom)
+		)
+	)
 	(label "LED"
 		(at 284.48 74.93 0)
@@
 		(unit 1)
 		(exclude_from_sim no)
-		(in_bom yes)
+		(in_bom no)
 		(on_board yes)
 		(dnp no)
-		(property "Reference" "Q2"
+		(property "Reference" "Q1"
 			(at 51.308 196.85 0)
 			(effects
@@
 			(project ""
 				(path "/9fde6b9c-53fd-4f64-9761-84b01b75f921"
-					(reference "Q2")
+					(reference "Q1")
 					(unit 1)
 				)
@@
 		(unit 1)
 		(exclude_from_sim no)
-		(in_bom yes)
+		(in_bom no)
 		(on_board yes)
 		(dnp no)
@@
 		(unit 1)
 		(exclude_from_sim no)
-		(in_bom yes)
+		(in_bom no)
 		(on_board yes)
 		(dnp no)
@@
 		(unit 1)
 		(exclude_from_sim no)
-		(in_bom yes)
+		(in_bom no)
 		(on_board yes)
 		(dnp no)
@@
 		(unit 1)
 		(exclude_from_sim no)
-		(in_bom yes)
+		(in_bom no)
 		(on_board yes)
 		(dnp no)
@@
 			)
 		)
-		(property "Footprint" "MountingHole:MountingHole_4.3mm_M4_DIN965"
+		(property "Footprint" "custom-parts:MountingHole_4.3mm_M4_Without-Screws"
 			(at 344.17 208.28 0)
 			(effects
@@
 		(dnp no)
 		(fields_autoplaced yes)
-		(property "Reference" "U3"
+		(property "Reference" "U2"
 			(at 120.65 33.02 0)
 			(effects
@@
 			(project ""
 				(path "/9fde6b9c-53fd-4f64-9761-84b01b75f921"
-					(reference "U3")
+					(reference "U2")
 					(unit 1)
 				)
@@
 		(unit 1)
 		(exclude_from_sim no)
-		(in_bom yes)
+		(in_bom no)
 		(on_board yes)
 		(dnp no)
@@
 		(unit 1)
 		(exclude_from_sim no)
-		(in_bom yes)
+		(in_bom no)
 		(on_board yes)
 		(dnp no)
@@
 			)
 		)
-		(property "Footprint" "Button_Switch_THT:SW_PUSH_6mm_H13mm"
+		(property "Footprint" "custom-parts:SW_PUSH_6mm_H13mm_No-Pad_Top-Left"
 			(at 186.69 252.73 0)
 			(effects
@@
 			)
 		)
-		(property "Footprint" "Rotary_Encoder:RotaryEncoder_Alps_EC12E_Vertical_H20mm"
+		(property "Footprint" "custom-parts:RotaryEncoder_Alps_EC12E_Vertical_H20mm_Mounting-Holes-GND"
 			(at 69.85 247.396 0)
 			(effects
@@
 		(unit 1)
 		(exclude_from_sim no)
-		(in_bom yes)
+		(in_bom no)
 		(on_board yes)
 		(dnp no)
@@
 		(unit 1)
 		(exclude_from_sim no)
-		(in_bom yes)
+		(in_bom no)
 		(on_board yes)
 		(dnp no)
@@
 		(unit 1)
 		(exclude_from_sim no)
-		(in_bom yes)
+		(in_bom no)
 		(on_board yes)
 		(dnp no)
@@
 		(unit 1)
 		(exclude_from_sim no)
-		(in_bom yes)
+		(in_bom no)
 		(on_board yes)
 		(dnp no)
@@
 		(unit 1)
 		(exclude_from_sim no)
-		(in_bom yes)
+		(in_bom no)
 		(on_board yes)
 		(dnp no)
@@
 		(unit 1)
 		(exclude_from_sim no)
-		(in_bom yes)
+		(in_bom no)
 		(on_board yes)
 		(dnp no)
@@
 			)
 		)
-		(property "Footprint" "MountingHole:MountingHole_4.3mm_M4"
+		(property "Footprint" "custom-parts:MountingHole_4.3mm_M4_Without-Screws"
 			(at 344.17 213.36 0)
 			(effects
@@
 		(unit 1)
 		(exclude_from_sim no)
-		(in_bom yes)
+		(in_bom no)
 		(on_board yes)
 		(dnp no)
@@
 			)
 		)
-		(property "Footprint" "Button_Switch_THT:SW_PUSH_6mm_H13mm"
+		(property "Footprint" "custom-parts:SW_PUSH_6mm_H13mm_No-Pad_Top-Right"
 			(at 127 252.73 0)
 			(effects
@@
 			)
 		)
-		(property "Footprint" "MountingHole:MountingHole_4.3mm_M4"
+		(property "Footprint" "custom-parts:MountingHole_4.3mm_M4_Without-Screws"
 			(at 349.25 208.28 0)
 			(effects
@@
 		(unit 1)
 		(exclude_from_sim no)
-		(in_bom yes)
+		(in_bom no)
 		(on_board yes)
 		(dnp no)
@@
 			)
 		)
-		(property "Footprint" "MountingHole:MountingHole_4.3mm_M4_DIN965"
+		(property "Footprint" "custom-parts:MountingHole_4.3mm_M4_Without-Screws"
 			(at 349.25 213.36 0)
 			(effects
@@
 		(unit 1)
 		(exclude_from_sim no)
-		(in_bom yes)
+		(in_bom no)
 		(on_board yes)
 		(dnp no)
@@
 			)
 		)
-		(property "Footprint" "Button_Switch_THT:SW_Slide_SPDT_Angled_CK_OS102011MA1Q"
+		(property "Footprint" "custom-parts:SW_Slide_SPDT_Angled_CK_OS102011MA1Q_Protruding"
 			(at 67.31 36.83 0)
 			(effects

Commit message: generate files for manufacturing
Parts:
- C1: LCSC Part Number (none) -> C19702
- C10, C11: LCSC Part Number (none) -> C1779
- C12, C13, C7: LCSC Part Number (none) -> C15195
- C14, C2, C3, C4, C5, C6: LCSC Part Number (none) -> C307331
- C15, C16, C17, C18, C8, C9: LCSC Part Number (none) -> C52923
- DFPlayerMini1: now left out of the parts list
- FB1: value 120R -> 600R; LCSC Part Number (none) -> C1002
- R1, R6, R7: LCSC Part Number (none) -> C25900
- R10, R11, R14, R16, R18, R2, R20, R8, R9: LCSC Part Number (none) -> C25744
- R12, R13: LCSC Part Number (none) -> C26083
- R15, R17, R19, R21: LCSC Part Number (none) -> C25768
- R22, R23, R4: LCSC Part Number (none) -> C25741
- R5: LCSC Part Number (none) -> C25076
- SW2: LCSC Part Number (none) -> C351238
- U1: LCSC Part Number (none) -> C8322
- U2: LCSC Part Number (none) -> C500795

Commit message: replace footprints with JLCs' footprints
Parts:
- SW2: footprint custom-parts:RotaryEncoder_Alps_EC12E_Vertical_H20mm_Mounting-Holes-GND -> custom-parts:SW-TH_EC12E24204A2
- U1: footprint Package_QFP:LQFP-64_10x10mm_P0.5mm -> custom-parts:LQFP-64_L10.0-W10.0-P0.50-LS12.0-BL
- U2: footprint Package_TO_SOT_SMD:SOT-223-3_TabPin2 -> custom-parts:SOT-223_L6.5-W3.5-P2.30-LS7.0-BR
Changed lines of the file:
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@@
 			)
 		)
-		(property "Footprint" "Package_TO_SOT_SMD:SOT-223-3_TabPin2"
+		(property "Footprint" "custom-parts:SOT-223_L6.5-W3.5-P2.30-LS7.0-BR"
 			(at 120.65 33.655 0)
 			(effects
 				(font
 					(size 1.27 1.27)
-					(italic yes)
 				)
 				(hide yes)
@@
 			)
 		)
-		(property "Footprint" "Package_QFP:LQFP-64_10x10mm_P0.5mm"
+		(property "Footprint" "custom-parts:LQFP-64_L10.0-W10.0-P0.50-LS12.0-BL"
 			(at 251.46 158.75 0)
 			(effects
@@
 			)
 		)
-		(property "Footprint" "custom-parts:RotaryEncoder_Alps_EC12E_Vertical_H20mm_Mounting-Holes-GND"
+		(property "Footprint" "custom-parts:SW-TH_EC12E24204A2"
 			(at 69.85 247.396 0)
 			(effects
